File: hardware/tokyo-metro-pcb.kicad_pcb (KiCad board)
At the start: 2 copper layers, 320 x 280 mm, 282 parts, among them SW1 TS-1187A-B-A-B, SW2 TS-1187A-B-A-B, SW3 TS-1187A-B-A-B, SW4 TS-1187A-B-A-B, U1 XIAO-RP2040-DIP

Commit message: Rebuild the KiCad board from the organic map
Placement, outline and artwork all come from the new input/tokyo.json:
248 LEDs at their stations, 13 row capacitors, the controller group at
(40, 220), and 1,555 route segments.

The route silkscreen is now cut around the label capsules and the LED
pads. tools/capsules.py holds that geometry and both preview_map and
export_art import it, rather than each keeping its own copy - every time
those two have had separate definitions they have drifted, and the
optimiser ends up solving a board nobody is drawing.

DRC: 2 shorts (mounting holes in the bay), 28 isolated copper islands and
16 starved thermals, all of which are the known front-pour-in-pieces
problem; schematic parity clean; 499 pads unconnected because nothing is
routed yet.

KNOWN GAP: the board draws its labels in KiCad's default stroke font,
while every label placement, capsule and collision check was computed
from Archivo Narrow SemiBold. The stroke font is 35-59% wider, so on the
board the names are wider than the space cleared for them. Either the
face has to be set on the text, or the layout has to be recomputed with
stroke-font metrics.

Co-Authored-By: Claude Opus 5 <noreply@anthropic.com>
Parts:
- moved LED205 236.8 mm to (101.1, 266.8)
- moved LED110 236.4 mm to (22.7, 21.2), turned to 90 degrees
- moved LED206 230.9 mm to (128.8, 264.1)
- moved LED207 225.4 mm to (147.7, 259.5)
- moved LED204 220.1 mm to (104.7, 251.9), turned to 90 degrees
- moved LED113 217.3 mm to (44.1, 61.6), turned to 180 degrees
- moved LED112 215.6 mm to (23.1, 53.9), turned to 180 degrees
- moved LED109 215.3 mm to (37.1, 32.3), turned to 0 degrees
- moved LED209 213.2 mm to (187.8, 246.9), turned to -90 degrees
- moved LED91 212.7 mm to (247.7, 14.0), turned to 90 degrees
- moved LED202 211.4 mm to (120.7, 244.0), turned to -45 degrees
- moved LED111 208.8 mm to (16.0, 46.2), turned to 180 degrees
- moved LED115 207.1 mm to (69.1, 52.4), turned to 180 degrees
- moved LED208 206.7 mm to (179.5, 240.7), turned to 180 degrees
- moved LED114 205.1 mm to (61.5, 76.7), turned to -90 degrees
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Other:
- board text added: "Akasaka-mitsuke"
- board text added: "Aoyama-itchome"
- board text added: "Arakawa-itchumae"
- board text added: "Arakawa-kuyakushomae"
- board text added: "Arakawa-nanachome"
- board text added: "Arakawa-nichome"
- board text added: "Arakawa-shakomae"
- board text added: "Arakawa-yuenchimae"
- board text added: "Ariake-Tennis-no-mori"
- board text added: "Higashi-ikebukuro"
- board text added: "Higashi-koenji"
- board text added: "Higashi-nakano"
- board text added: "Higashi-nihombashi"
- board text added: "Higashi-ogu-sanchome"
- board text added: "Higashi-shinjuku"
- board text added: "Hongo-sanchome"
- board text added: "Honjo-azumabashi"
- board text added: "Itabashi-kuyakushomae"
- board text added: "Kiyosumi-shirakawa"
- board text added: "Kokkai-gijidomae"
- board text added: "Kokuritsu-kyogijo"
- board text added: "Kokusai-tenjijo"
- board text added: "Kotake-mukaihara"
- board text added: "Machiya-ekimae"
- board text added: "Machiya-nichome"
- board text added: "Meiji-jingumae"
- board text added: "Minami-sunamachi"
- board text added: "Monzen-nakacho"
- board text added: "Naka-okachimachi"
- board text added: "Nakano-fujimicho"
- board text added: "Nakano-shimbashi"
- board text added: "Nishi-shinjuku"
- board text added: "Nishi-shinjuku-gochome"
- board text added: "Nishigahara-yonchome"
- board text added: "Ochiai-minami-nagasaki"
- board text added: "Odaiba-kaihinkoen"
- board text added: "Roppongi-itchome"
- board text added: "Shin-koshinzuka"
- board text added: "Shin-ochanomizu"
- board text added: "Shin-okachimachi"
- board text added: "Shinjuku-gyoemmae"
- board text added: "Shinjuku-nishiguchi"
- board text added: "Shinjuku-sanchome"
- board text added: "Shirokane-takanawa"
- board text added: "Takinogawa-itchome"
- board text added: "Toden-zoshigaya"
- board text added: "Ueno-okachimachi"
- board text added: "Ushigome-kagurazaka"
- board text added: "Ushigome-yanagicho"
- board text added: "Wakamatsu-kawada"
- board text added: "Yotsuya-sanchome"
- board text removed: "Akasaka mitsuke"
- board text removed: "Aoyama itchome"
- board text removed: "Arakawa itchumae"
- board text removed: "Arakawa kuyakushomae"
- board text removed: "Arakawa nanachome"
- board text removed: "Arakawa nichome"
- board text removed: "Arakawa shakomae"
- board text removed: "Arakawa yuenchimae"
- board text removed: "Ariake Tennis-no-mori"
- board text removed: "Higashi ikebukuro"
- board text removed: "Higashi koenji"
- board text removed: "Higashi nakano"
- board text removed: "Higashi nihombashi"
- board text removed: "Higashi ogu-sanchome"
- board text removed: "Higashi shinjuku"
- board text removed: "Hongo sanchome"
- board text removed: "Honjo azumabashi"
- board text removed: "Itabashi kuyakushomae"
- board text removed: "Kiyosumi shirakawa"
- board text removed: "Kokkai gijidomae"
- board text removed: "Kokuritsu kyogijo"
- board text removed: "Kokusai tenjijo"
- board text removed: "Kotake mukaihara"
- board text removed: "Machiya ekimae"
- board text removed: "Machiya nichome"
- board text removed: "Meiji jingumae"
- board text removed: "Minami sunamachi"
- board text removed: "Monzen nakacho"
- board text removed: "Naka okachimachi"
- board text removed: "Nakano fujimicho"
- board text removed: "Nakano shimbashi"
- board text removed: "Nishi shinjuku"
- board text removed: "Nishi shinjuku-gochome"
- board text removed: "Nishigahara yonchome"
- board text removed: "Ochiai minami-nagasaki"
- board text removed: "Odaiba kaihinkoen"
- board text removed: "Roppongi itchome"
- board text removed: "Shin koshinzuka"
- board text removed: "Shin ochanomizu"
- board text removed: "Shin okachimachi"
- board text removed: "Shinjuku gyoemmae"
- board text removed: "Shinjuku nishiguchi"
- board text removed: "Shinjuku sanchome"
- board text removed: "Shirokane takanawa"
- board text removed: "Takinogawa itchome"
- board text removed: "Toden zoshigaya"
- board text removed: "Ueno okachimachi"
- board text removed: "Ushigome kagurazaka"
- board text removed: "Ushigome yanagicho"
- board text removed: "Wakamatsu kawada"
- board text removed: "Yotsuya sanchome"
