File: hardware/tokyo-metro-pcb.kicad_pcb (KiCad board)
At the start: 2 copper layers, 320 x 280 mm, 282 parts, among them SW1 TS-1187A-B-A-B, SW2 TS-1187A-B-A-B, SW3 TS-1187A-B-A-B, SW4 TS-1187A-B-A-B, U1 XIAO-RP2040-DIP

Commit message: Every LED pin 1 up, and a polarity mark that can be read
Pads 1 and 4 of the XL-1615 sit on the SAME edge of the part, so a part
fitted 180 degrees out swaps GND with DI and +5V with DO. The vendor's
silk dot was on pad 1's side but centred between the two pads: it marked
the side and nothing more. It now sits on pad 1's row, 0.750 mm from
pad 1 and 1.172 from pad 4 on all 248, in the project library as well as
on the board so the two agree. F.Fab was already unambiguous.

The LEDs were each turned so DOUT faced the next station - eight angles
across the board, which is right if the router is what you optimise and
wrong for whoever fits 248 parts. All 248 are at 270 degrees now, pin 1
up, with the dot directly above it. Routing gets harder; assembly
becomes checkable in one glance, and in one photograph.

Being geometrically right was not enough. The dot is white silk in a map
made of white silk, and with the ring at 1.65 its band ran through the
dot on every LED - not one of the 248 had half its ink standing clear.
Cutting the dot out of the routes and notching it out of the ring takes
that to 184 fully clear and 190 at 90% or better. The ring still reads
as a circle and the notch is at pin 1, which is a second cue for free.
Thirteen dots are still under a station name's glyphs; the label
optimiser does not know the dots exist.

pad_to_mask_clearance was 0.2 mm with no footprint override, so each
0.8 mm pad got a 1.2 mm opening and the 0.25 mm pad-to-pad gaps vanished
entirely - 199 solder_mask_bridge warnings, on a check the project had
set to "ignore". At the standard 0.05 the dams come out at 0.150 mm,
which JLCPCB makes in any colour at 1 oz. Three stacked GND zones with
byte-identical outlines are down to one; their slivers accounted for all
32 isolated_copper reports.

The back carried a Montreal Metro credit with the Montreal repo URL, and
an owl. Both gone.

DRC: 0 shorts, 0 clearance, 0 isolated copper, 0 mask bridges, 0 parity.
Left are 16 starved thermal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
Parts:
- removed LOGO1: artwork, 
- added ROW13: 1uF,16V,X5R, Capacitor_SMD:C_0402_1005Metric, F.Cu at (164.5, 50.9)
- added ROW14: 1uF,16V,X5R, Capacitor_SMD:C_0402_1005Metric, F.Cu at (210.4, 62.0)
- added ROW15: 1uF,16V,X5R, Capacitor_SMD:C_0402_1005Metric, F.Cu at (169.8, 89.7)
- added ROW16: 1uF,16V,X5R, Capacitor_SMD:C_0402_1005Metric, F.Cu at (129.9, 59.7)
- added ROW17: 1uF,16V,X5R, Capacitor_SMD:C_0402_1005Metric, F.Cu at (146.2, 28.8)
- added ROW18: 1uF,16V,X5R, Capacitor_SMD:C_0402_1005Metric, F.Cu at (184.9, 48.5)
- added ROW19: 1uF,16V,X5R, Capacitor_SMD:C_0402_1005Metric, F.Cu at (182.6, 46.7)
- added ROW20: 1uF,16V,X5R, Capacitor_SMD:C_0402_1005Metric, F.Cu at (128.9, 24.9)
- added ROW21: 1uF,16V,X5R, Capacitor_SMD:C_0402_1005Metric, F.Cu at (118.0, 43.9)
- added ROW22: 1uF,16V,X5R, Capacitor_SMD:C_0402_1005Metric, F.Cu at (56.1, 47.2)
- added ROW23: 1uF,16V,X5R, Capacitor_SMD:C_0402_1005Metric, F.Cu at (44.1, 64.6)
- added ROW24: 1uF,16V,X5R, Capacitor_SMD:C_0402_1005Metric, F.Cu at (88.7, 80.0)
- added ROW25: 1uF,16V,X5R, Capacitor_SMD:C_0402_1005Metric, F.Cu at (80.5, 112.0)
- added ROW26: 1uF,16V,X5R, Capacitor_SMD:C_0402_1005Metric, F.Cu at (116.8, 118.0)
- added ROW27: 1uF,16V,X5R, Capacitor_SMD:C_0402_1005Metric, F.Cu at (101.2, 77.7)
- added ROW28: 1uF,16V,X5R, Capacitor_SMD:C_0402_1005Metric, F.Cu at (111.5, 70.0)
- added ROW29: 1uF,16V,X5R, Capacitor_SMD:C_0402_1005Metric, F.Cu at (116.3, 83.4)
- added ROW30: 1uF,16V,X5R, Capacitor_SMD:C_0402_1005Metric, F.Cu at (133.6, 114.4)
- added ROW31: 1uF,16V,X5R, Capacitor_SMD:C_0402_1005Metric, F.Cu at (92.0, 132.7)
- added ROW32: 1uF,16V,X5R, Capacitor_SMD:C_0402_1005Metric, F.Cu at (64.5, 127.3)
- added ROW33: 1uF,16V,X5R, Capacitor_SMD:C_0402_1005Metric, F.Cu at (64.0, 102.3)
- added ROW34: 1uF,16V,X5R, Capacitor_SMD:C_0402_1005Metric, F.Cu at (56.5, 167.0)
- added ROW35: 1uF,16V,X5R, Capacitor_SMD:C_0402_1005Metric, F.Cu at (89.5, 160.9)
- added ROW36: 1uF,16V,X5R, Capacitor_SMD:C_0402_1005Metric, F.Cu at (117.9, 170.8)
- added ROW37: 1uF,16V,X5R, Capacitor_SMD:C_0402_1005Metric, F.Cu at (141.5, 181.2)
- added ROW38: 1uF,16V,X5R, Capacitor_SMD:C_0402_1005Metric, F.Cu at (145.3, 159.9)
- added ROW39: 1uF,16V,X5R, Capacitor_SMD:C_0402_1005Metric, F.Cu at (136.1, 141.0)
- added ROW40: 1uF,16V,X5R, Capacitor_SMD:C_0402_1005Metric, F.Cu at (141.7, 158.8)
- added ROW41: 1uF,16V,X5R, Capacitor_SMD:C_0402_1005Metric, F.Cu at (100.8, 221.0)
- added ROW42: 1uF,16V,X5R, Capacitor_SMD:C_0402_1005Metric, F.Cu at (101.7, 251.9)
- added ROW43: 1uF,16V,X5R, Capacitor_SMD:C_0402_1005Metric, F.Cu at (176.5, 240.7)
- added ROW44: 1uF,16V,X5R, Capacitor_SMD:C_0402_1005Metric, F.Cu at (181.9, 236.2)
- added ROW45: 1uF,16V,X5R, Capacitor_SMD:C_0402_1005Metric, F.Cu at (125.2, 206.0)
- added ROW46: 1uF,16V,X5R, Capacitor_SMD:C_0402_1005Metric, F.Cu at (157.5, 197.7)
- added ROW47: 1uF,16V,X5R, Capacitor_SMD:C_0402_1005Metric, F.Cu at (168.3, 170.7)
- added ROW48: 1uF,16V,X5R, Capacitor_SMD:C_0402_1005Metric, F.Cu at (177.0, 143.0)
- added ROW49: 1uF,16V,X5R, Capacitor_SMD:C_0402_1005Metric, F.Cu at (189.0, 126.8)
- added ROW50: 1uF,16V,X5R, Capacitor_SMD:C_0402_1005Metric, F.Cu at (250.1, 134.2)
- added ROW51: 1uF,16V,X5R, Capacitor_SMD:C_0402_1005Metric, F.Cu at (293.1, 174.2)
- ROW0, ROW1, ROW10, ROW11, ROW12, ROW2, ROW3, ROW4, ROW5, ROW6, ROW7, ROW8, ROW9: value 10uF,10V,X5R -> 1uF,16V,X5R
- moved ROW5 164.9 mm to (163.8, 161.2)
- moved ROW8 138.6 mm to (166.5, 116.8)
- moved ROW10 135.9 mm to (170.2, 99.6)
- moved ROW4 132.4 mm to (181.9, 167.3), turned to 0 degrees
- moved ROW11 120.9 mm to (220.7, 103.3)
- moved ROW2 83.5 mm to (241.1, 164.9)
- moved ROW3 83.2 mm to (216.4, 144.4)
- moved ROW1 67.5 mm to (199.8, 201.5), turned to 0 degrees
- moved ROW9 58.7 mm to (182.4, 127.4), turned to 0 degrees
- moved ROW6 50.3 mm to (160.6, 135.4), turned to 90 degrees
- moved ROW12 44.0 mm to (192.1, 92.8)
- moved ROW7 34.5 mm to (157.7, 104.9), turned to 0 degrees
- moved ROW0 29.1 mm to (219.7, 212.6)
- turned LED1 to -90 degrees
- turned LED10 to -90 degrees
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Connections:
- R1 pad 1: unconnected-(R1-Pad1) -> LED_DATA
- R1 pad 2: unconnected-(R1-Pad2) -> LED_IN
Other:
- rule pad_to_mask_clearance: 0.2 -> 0.05
- board text added: "Tokyo Metro Github.com/Funvill/tokyo-metro-pcb Version: 2026-Oct"
- board text removed: "Montréal Métro Github.com/Funvill/montreal-skytrain-pcb Version: 2026-Oct"
