File: hardware/tokyo-metro-pcb.kicad_pcb (KiCad board)
At the start: 2 copper layers, 320 x 280 mm, 320 parts, among them SW1 TS-1187A-B-A-B, SW2 TS-1187A-B-A-B, SW3 TS-1187A-B-A-B, SW4 TS-1187A-B-A-B, U1 XIAO-RP2040-DIP

Commit message: Autoroute the chain, and take out the copper that connects nothing
Planes on both layers: +5V on the front, GND on the back, with the
back-side hardware in a row along the bottom edge and the XIAO 40 mm up
from it so the cable has somewhere to go. The Power net class widens to
0.8 mm.

Freerouting took the data chain from 863 unrouted down to 34. Importing
the result left a lot of copper behind that was not carrying anything:

  - 116 vias with nothing on the far end
  - 67 track stubs, which only appeared as the vias came out - the
    pattern was pad -> short track -> via -> nothing, so removing a via
    turned its track into the dangling item and exposed the one behind
    it. Four rounds to exhaust the chains.
  - the vestigial gnd_back zone, 239 mm square, left from when both
    layers were ground

Matching report items to board objects is the part worth being careful
about. A track's GetPosition() is its START, not the end the report
names, and those coincide with via positions - matching on position
alone removed 240 objects for 112 reported items and broke real
connections. Match on net, layer, length and one of the two ENDS. The
last five were mirrored pairs sharing all four, two tracks of equal
length radiating from one point; they separate on the far end, where one
continues into the route and the other stops in air.

Unconnected items stayed at 34 through every removal, which is the
number that says this took out copper that was connecting nothing.

DRC: via_dangling 116 -> 0, track_dangling 32 -> 0, isolated_copper
23 -> 0, parity 0. What is left is 12 clearance grazes, 74 starved
thermals on pads inside the pour, and the 11 silk_edge_clearance
warnings the station names near the border have always raised.

Co-Authored-By: Claude Opus 5 <noreply@anthropic.com>
Parts:
- moved +5V1 287.7 mm to (145.0, 270.0)
- moved LED_OUT1 162.0 mm to (135.0, 270.0)
- moved TP4 150.9 mm to (120.0, 270.0)
- moved TP3 143.3 mm to (110.0, 270.0)
- moved TP2 136.0 mm to (100.0, 270.0)
- moved TP1 129.8 mm to (90.0, 270.0)
- moved +5V2 20.0 mm to (46.0, 259.0)
- moved C1 20.0 mm to (48.0, 216.0)
- moved GND1 20.0 mm to (40.0, 259.0)
- moved LED_IN1 20.0 mm to (34.0, 259.0)
- moved R1 20.0 mm to (34.0, 216.0)
- moved SW1 20.0 mm to (22.0, 228.0)
- moved SW2 20.0 mm to (22.0, 252.0)
- moved SW3 20.0 mm to (58.0, 228.0)
- moved SW4 20.0 mm to (58.0, 252.0)
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Routing:
- net +5V: track 0.00 -> 3475.1 mm, vias 0 -> 145
- net GND: track 0.00 -> 311.5 mm, vias 0 -> 169
- net BUTTON_04: track 0.00 -> 126.5 mm, vias 0 -> 3
- net BUTTON_03: track 0.00 -> 115.0 mm, vias 0 -> 2
- net BUTTON_01: track 0.00 -> 112.8 mm, vias 0 -> 2
- net Net-(LED90-DO): track 0.00 -> 65.8 mm, vias 0 -> 2
- net LED_DATA: track 0.00 -> 62.1 mm, vias 0 -> 1
- net BUTTON_02: track 0.00 -> 61.1 mm
- net Net-(LED107-DO): track 0.00 -> 48.5 mm
- net Net-(LED241-DO): track 0.00 -> 47.0 mm, vias 0 -> 2
- net Net-(LED165-DO): track 0.00 -> 46.1 mm, vias 0 -> 2
- net Net-(LED92-DO): track 0.00 -> 41.5 mm, vias 0 -> 2
- net Net-(LED247-DO): track 0.00 -> 41.0 mm, vias 0 -> 2
- net Net-(LED91-DO): track 0.00 -> 39.8 mm, vias 0 -> 2
- net Net-(LED97-DO): track 0.00 -> 39.3 mm, vias 0 -> 2
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