File: hardware/tokyo-metro-pcb.kicad_sch (KiCad schematic)
At the start: 281 parts, among them SW1 TS-1187A-B-A-B, SW2 TS-1187A-B-A-B, SW3 TS-1187A-B-A-B, SW4 TS-1187A-B-A-B, U1 XIAO-RP2040-DIP

Commit message: Reconnect R1, and make the checks assert what they only printed
make_schematic.py deleted the LED_DATA and LED_IN global labels off R1's
two pins and never inserted the replacement wire+label blocks it had
built: it appended `gen` and dropped `tidy`. GPIO1 dead-ended at its test
point, both of R1's pads fell to unconnected-(R1-Pad*), and LED1's DI sat
alone on a one-node net. The chain itself was continuous end to end,
which is all check_led_chain.py asserted, so every check passed on a
board where not one LED would have lit.

The replacement blocks were wrong as well, and nobody could see it
because they were never rendered. For a vertical schematic label the
angle does not choose which side of the anchor the text sits on - KiCad
always sets vertical text bottom-to-top, so 90 and 270 put the glyphs on
the same side and only the justify moves them. Both labels ran their
text back across the resistor. check_schematic.py derived the box from
the angle, so it modelled LED_IN as running down into empty space while
it actually ran up into R1's body, and reported 0 overlapping pairs on a
sheet that had one. LED_IN was the only 90-degree label on the sheet.

Decoupling goes from 13 caps to 52, four per row, and from 10uF,10V,X5R
in an 0402 - not a part that exists to buy - to 1uF,16V,X5R. One cap per
row of 20 LEDs is bulk, not decoupling: the far LED sat nineteen pitches
of trace from it. This took three tries, each silent. The caps' Value
text is 11.3 mm wide and collided with the LEDs, so they moved to the
clear band right of each row. The power rail still stopped at the last
LED, so all 39 new caps floated with both pads unconnected. Extending
the rail then turned the last LED's stub from an end-to-end meeting into
a tee, and in KiCad a wire ending mid-wire is not connected without an
explicit junction, so one LED per row went dark too.

check_led_chain.py now walks the head of the chain to a controller pin,
requires each rail to reach the controller rather than merely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
Parts:
- added ROW13, ROW14, ROW15, ROW16, ROW17, ROW18, ROW19, ROW20, ROW21, ROW22, ROW23, ROW24, ROW25, ROW26, ROW27, ROW28, ROW29, ROW30, ROW31, ROW32, ROW33, ROW34, ROW35, ROW36, ROW37, ROW38, ROW39, ROW40, ROW41, ROW42, ROW43, ROW44, ROW45, ROW46, ROW47, ROW48, ROW49, ROW50, ROW51: 1uF,16V,X5R, Capacitor_SMD:C_0402_1005Metric, symbol __sws_jlpcb:jlcpcb-1uF,25V,X5R
- ROW0, ROW1, ROW10, ROW11, ROW12, ROW2, ROW3, ROW4, ROW5, ROW6, ROW7, ROW8, ROW9: value 10uF,10V,X5R -> 1uF,16V,X5R
Connections:
- net +5V: now also ROW13.2, ROW14.2, ROW15.2, ROW16.2, ROW17.2, ROW18.2, ROW19.2, ROW20.2, ROW21.2, ROW22.2, ROW23.2, ROW24.2, ROW25.2, ROW26.2, ROW27.2, ROW28.2, ROW29.2, ROW30.2, ROW31.2, ROW32.2, ROW33.2, ROW34.2, ROW35.2, ROW36.2, ROW37.2, ROW38.2, ROW39.2, ROW40.2, ROW41.2, ROW42.2, ROW43.2, ROW44.2, ROW45.2, ROW46.2, ROW47.2, ROW48.2, ROW49.2, ROW50.2, ROW51.2
- net GND: now also ROW13.1, ROW14.1, ROW15.1, ROW16.1, ROW17.1, ROW18.1, ROW19.1, ROW20.1, ROW21.1, ROW22.1, ROW23.1, ROW24.1, ROW25.1, ROW26.1, ROW27.1, ROW28.1, ROW29.1, ROW30.1, ROW31.1, ROW32.1, ROW33.1, ROW34.1, ROW35.1, ROW36.1, ROW37.1, ROW38.1, ROW39.1, ROW40.1, ROW41.1, ROW42.1, ROW43.1, ROW44.1, ROW45.1, ROW46.1, ROW47.1, ROW48.1, ROW49.1, ROW50.1, ROW51.1
- net LED_DATA: now also R1.1
- net LED_IN: now also R1.2
Other:
- moved on the sheet: ROW1, ROW10, ROW11, ROW12, ROW2, ROW3, ROW4, ROW5, ROW6, ROW7, ROW8, ROW9
